Commit message: bug fixes

File: src/arm_model/description/urdf/arm_model.urdf.xacro (robot description, xacro)
@@ -12,5 +12,5 @@
   <xacro:include filename="arm_model.materials.xacro" />
   <!-- Import arm_model ros2_control description -->
-  <xacro:include filename="$(find description)/ros2_control/arm_model.ros2_control.xacro" />
+  <xacro:include filename="$(find arm_model)/description/ros2_control/arm_model.ros2_control.xacro"/>
   <!-- Used for fixing robot -->
   <link name="world"/>

File: src/arm_model/description/urdf/arm_model_description.urdf.xacro (robot description, xacro)
@@ -102,3 +102,4 @@
       <origin xyz="0 0 ${arm_length}"/>
     </joint>
-    robot>
+  </xacro:macro>
+</robot>
